Commit message: Working custom contact plan on stepping stones.

File: project/robots/unitree_go2/urdf/go2_description.urdf (robot description, URDF)
Before this commit: robot go2_description, 29 links, 28 joints
Links:
- link FL_thigh: geometry collision box size=0.11 0.0245 0.034; visual mesh filename=package://dae/thigh.dae
- link FR_thigh: geometry collision box size=0.11 0.0245 0.034; visual mesh filename=package://dae/thigh_mirror.dae
- link RL_thigh: geometry collision box size=0.11 0.0245 0.034; visual mesh filename=package://dae/thigh.dae
- link RR_thigh: geometry collision box size=0.11 0.0245 0.034; visual mesh filename=package://dae/thigh_mirror.dae
